File: hardware/auto-garden/auto-garden.sch (KiCad schematic (older format))
At the start: 2 parts

Commit message: Finished KiCAD schematic and annotation
Parts:
- removed U?: LM1085-5.0, symbol Regulator_Linear:LM1085-5.0
- removed U?: MCP1702-3302E_TO92-3, Package_TO_SOT_SMD:SOT-89-3, symbol auto-garden:MCP1702-3302E_TO92-3
- added C1, C10, C3, C5, C6, C9: 0.1u, symbol Device:C
- added C11, C2, C4, C7, C8: 0.001u, symbol Device:C
- added J1, J5: Conn_01x02_Female, symbol Connector:Conn_01x02_Female
- added J2: Conn_01x06_Female, symbol Connector:Conn_01x06_Female
- added J3, J4: Conn_01x03_Female, symbol Connector:Conn_01x03_Female
- added J6: USB_A, symbol Connector:USB_A
- added JP1, JP2: Jumper_2_Open, symbol Jumper:Jumper_2_Open
- added Q1, Q3: Q_PMOS_DGS, symbol Device:Q_PMOS_DGS
- added Q2, Q4: Q_NMOS_DGS, symbol Device:Q_NMOS_DGS
- added R1, R2, R3: 5k, symbol Device:R
- added R4: 27, symbol Device:R
- added R5: 10, symbol Device:R
- added U1: AP2127R-3.3, Package_TO_SOT_SMD:SOT-89-3, symbol auto-garden:AP2127R-3.3
- added U2: MCP3001, Package_DIP:DIP-8_W7.62mm, symbol auto-garden:MCP3001
Connections:
- net +3V3: now also C10.1, C11.1, C3.1, C4.1, C5.1, C6.1, C7.1, C8.1, C9.1, J3.2 (Pin_2), J4.1 (Pin_1), R1.1, U1.3 (VO), U2.1 (VREF), U2.8 (VDD)
- net +5V: now also C1.1, C2.1, J1.2 (Pin_2), Q1.1 (D), Q3.1 (D), U1.2 (VI)
- net GND: now also C1.2, C10.2, C11.2, C2.2, C3.2, C4.2, C5.2, C6.2, C7.2, C8.2, C9.2, J1.1 (Pin_1), J3.3 (Pin_3), J4.3 (Pin_3), J5.2 (Pin_2), J6.4 (GND), J6.5 (Shield), Q2.3 (S), Q4.3 (S), R2.1, R3.1, U1.1 (GND), U2.3 (IN-), U2.4 (VSS)
- new net: JP1.1 (A), Q1.3 (S), Q2.1 (D), R4.2
- new net: J5.1 (Pin_1), JP1.2 (B), R4.1
- new net: JP2.1 (A), Q3.3 (S), Q4.1 (D), R5.2
- new net: J6.1 (VBUS), JP2.2 (B), R5.1
- new net: J3.1 (Pin_1), U2.2 (IN+)
- new net P2: J2.2 (Pin_2), J4.2 (Pin_2), R1.2
- new net P3_CLK: J2.3 (Pin_3), U2.7 (CLK)
- new net P4_data: J2.4 (Pin_4), U2.6 (D_out)
- new net P5_~CS: J2.5 (Pin_5), U2.5 (~CS)
- new net ~P1: J2.1 (Pin_1), Q1.2 (G), Q2.2 (G), R2.2
- new net ~P6: J2.6 (Pin_6), Q3.2 (G), Q4.2 (G), R3.2
- no-connect marks 0 -> 2
Other:
- note added: "DHT11"
- note added: "External Power In"
- note added: "Moisture Sensor"
- note added: "Motor"

Commit message: Finished schematic
Parts:
- removed J4: Conn_01x03_Female, symbol Connector:Conn_01x03_Female
- removed J5: Conn_01x02_Female, symbol Connector:Conn_01x02_Female
- removed J6: USB_A, symbol Connector:USB_A
- added J4: Conn_01x03_Male, Connector_PinHeader_1.27mm:PinHeader_1x03_P1.27mm_Vertical, symbol Connector:Conn_01x03_Male
- added J5, J6: Screw_Terminal_01x02, auto-garden:Phoenix Contact COMBICON PTSA, symbol Connector:Screw_Terminal_01x02
- C1, C10, C3, C5, C6, C9: footprint (none) -> Capacitor_THT:C_Rect_L4.0mm_W2.5mm_P2.50mm
- C11, C2, C4, C7, C8: footprint (none) -> Capacitor_THT:C_Disc_D5.0mm_W2.5mm_P5.00mm
- J1: footprint (none) -> Connector_PinHeader_1.27mm:PinHeader_1x02_P1.27mm_Vertical
- J2: footprint (none) -> Connector_PinHeader_1.27mm:PinHeader_1x06_P1.27mm_Vertical
- J3: footprint (none) -> Connector_PinHeader_1.27mm:PinHeader_1x03_P1.27mm_Vertical
- JP1, JP2: footprint (none) -> Jumper:SolderJumper-2_P1.3mm_Open_RoundedPad1.0x1.5mm
- Q1, Q2, Q3, Q4: footprint (none) -> Package_TO_SOT_THT:TO-92
- R1, R2, R3, R4, R5: footprint (none) -> Resistor_THT:R_Axial_DIN0207_L6.3mm_D2.5mm_P10.16mm_Horizontal
Connections:
- net +3V3: now also J4.1 (Pin_1)
- net GND: now also J4.3 (Pin_3), J5.2 (Pin_2), J6.2 (Pin_2)
- net P2: now also J4.2 (Pin_2)
- net at JP1.2 (B), R4.1: now also J5.1 (Pin_1)
- net at JP2.2 (B), R5.1: now also J6.1 (Pin_1)
- no-connect marks 2 -> 0
Other:
- note added: "USB LED"
Changed lines of the file:
@@
 Sheet 1 1
 Title "Auto-Garden-Top-Level"
-Date "2019-08-27"
-Rev "0.1"
+Date "2019-10-27"
+Rev "1.0"
 Comp "SouderFamily"
 Comment1 ""
@@
 F 0 "Q1" H 8656 2146 50  0000 L CNN
 F 1 "Q_PMOS_DGS" H 8656 2055 50  0000 L CNN
-F 2 "" H 8650 2200 50  0001 C CNN
+F 2 "Package_TO_SOT_THT:TO-92" H 8650 2200 50  0001 C CNN
 F 3 "~" H 8450 2100 50  0001 C CNN
 	1    8450 2100
@@
 F 0 "Q2" H 8656 2646 50  0000 L CNN
 F 1 "Q_NMOS_DGS" H 8656 2555 50  0000 L CNN
-F 2 "" H 8650 2700 50  0001 C CNN
+F 2 "Package_TO_SOT_THT:TO-92" H 8650 2700 50  0001 C CNN
 F 3 "~" H 8450 2600 50  0001 C CNN
 	1    8450 2600
@@
 F 0 "R4" V 9343 2350 50  0000 C CNN
 F 1 "27" V 9434 2350 50  0000 C CNN
-F 2 "" V 9480 2350 50  0001 C CNN
+F 2 "Resistor_THT:R_Axial_DIN0207_L6.3mm_D2.5mm_P10.16mm_Horizontal" V 9480 2350 50  0001 C CNN
 F 3 "~" H 9550 2350 50  0001 C CNN
 	1    9550 2350
@@
 F 0 "JP1" H 9550 2475 50  0000 C CNN
 F 1 "Jumper_2_Open" H 9550 2566 50  0000 C CNN
-F 2 "" H 9550 2700 50  0001 C CNN
+F 2 "Jumper:SolderJumper-2_P1.3mm_Open_RoundedPad1.0x1.5mm" H 9550 2700 50  0001 C CNN
 F 3 "~" H 9550 2700 50  0001 C CNN
 	1    9550 2700
@@
 F 0 "R2" H 7980 2554 50  0000 R CNN
 F 1 "5k" H 7980 2645 50  0000 R CNN
-F 2 "" V 7980 2600 50  0001 C CNN
+F 2 "Resistor_THT:R_Axial_DIN0207_L6.3mm_D2.5mm_P10.16mm_Horizontal" V 7980 2600 50  0001 C CNN
 F 3 "~" H 8050 2600 50  0001 C CNN
 	1    8050 2600
@@
 F 0 "Q3" H 8806 4346 50  0000 L CNN
 F 1 "Q_PMOS_DGS" H 8806 4255 50  0000 L CNN
-F 2 "" H 8800 4400 50  0001 C CNN
+F 2 "Package_TO_SOT_THT:TO-92" H 8800 4400 50  0001 C CNN
 F 3 "~" H 8600 4300 50  0001 C CNN
 	1    8600 4300
@@
 F 0 "Q4" H 8806 4846 50  0000 L CNN
 F 1 "Q_NMOS_DGS" H 8806 4755 50  0000 L CNN
-F 2 "" H 8800 4900 50  0001 C CNN
+F 2 "Package_TO_SOT_THT:TO-92" H 8800 4900 50  0001 C CNN
 F 3 "~" H 8600 4800 50  0001 C CNN
 	1    8600 4800
@@
 F 0 "R5" V 9493 4550 50  0000 C CNN
 F 1 "10" V 9584 4550 50  0000 C CNN
-F 2 "" V 9630 4550 50  0001 C CNN
+F 2 "Resistor_THT:R_Axial_DIN0207_L6.3mm_D2.5mm_P10.16mm_Horizontal" V 9630 4550 50  0001 C CNN
 F 3 "~" H 9700 4550 50  0001 C CNN
 	1    9700 4550
@@
 F 0 "JP2" H 9700 4675 50  0000 C CNN
 F 1 "Jumper_2_Open" H 9700 4766 50  0000 C CNN
-F 2 "" H 9700 4900 50  0001 C CNN
+F 2 "Jumper:SolderJumper-2_P1.3mm_Open_RoundedPad1.0x1.5mm" H 9700 4900 50  0001 C CNN
 F 3 "~" H 9700 4900 50  0001 C CNN
 	1    9700 4900
@@
 F 0 "R3" H 8130 4754 50  0000 R CNN
 F 1 "5k" H 8130 4845 50  0000 R CNN
-F 2 "" V 8130 4800 50  0001 C CNN
+F 2 "Resistor_THT:R_Axial_DIN0207_L6.3mm_D2.5mm_P10.16mm_Horizontal" V 8130 4800 50  0001 C CNN
 F 3 "~" H 8200 4800 50  0001 C CNN
 	1    8200 4800
@@
 	8200 4550 7950 4550
 Connection ~ 8200 4550
-$Comp
-L Connector:Conn_01x03_Female J4
-U 1 1 5DB7B0A5
-P 5800 2850
-F 0 "J4" H 5828 2876 50  0000 L CNN
-F 1 "Conn_01x03_Female" H 5828 2785 50  0000 L CNN
-F 2 "" H 5800 2850 50  0001 C CNN
-F 3 "~" H 5800 2850 50  0001 C CNN
-	1    5800 2850
-	1    0    0    -1
-$EndComp
 Text Notes 5950 2850 0    50   ~ 0
 DHT11
@@
 F 0 "C9" H 4965 2396 50  0000 L CNN
 F 1 "0.1u" H 4965 2305 50  0000 L CNN
-F 2 "" H 4888 2200 50  0001 C CNN
+F 2 "Capacitor_THT:C_Rect_L4.0mm_W2.5mm_P2.50mm" H 4888 2200 50  0001 C CNN
 F 3 "~" H 4850 2350 50  0001 C CNN
 	1    4850 2350
@@
 F 0 "R1" H 5370 2596 50  0000 L CNN
 F 1 "5k" H 5370 2505 50  0000 L CNN
-F 2 "" V 5230 2550 50  0001 C CNN
+F 2 "Resistor_THT:R_Axial_DIN0207_L6.3mm_D2.5mm_P10.16mm_Horizontal" V 5230 2550 50  0001 C CNN
 F 3 "~" H 5300 2550 50  0001 C CNN
 	1    5300 2550
@@
 F 0 "C10" H 6465 4046 50  0000 L CNN
 F 1 "0.1u" H 6465 3955 50  0000 L CNN
-F 2 "" H 6388 3850 50  0001 C CNN
+F 2 "Capacitor_THT:C_Rect_L4.0mm_W2.5mm_P2.50mm" H 6388 3850 50  0001 C CNN
 F 3 "~" H 6350 4000 50  0001 C CNN
 	1    6350 4000
@@
 F 0 "C11" H 6865 4046 50  0000 L CNN
 F 1 "0.001u" H 6865 3955 50  0000 L CNN
-F 2 "" H 6788 3850 50  0001 C CNN
+F 2 "Capacitor_THT:C_Disc_D5.0mm_W2.5mm_P5.00mm" H 6788 3850 50  0001 C CNN
 F 3 "~" H 6750 4000 50  0001 C CNN
 	1    6750 4000
@@
 F 0 "C8" H 4815 4146 50  0000 L CNN
 F 1 "0.001u" H 4815 4055 50  0000 L CNN
-F 2 "" H 4738 3950 50  0001 C CNN
+F 2 "Capacitor_THT:C_Disc_D5.0mm_W2.5mm_P5.00mm" H 4738 3950 50  0001 C CNN
 F 3 "~" H 4700 4100 50  0001 C CNN
 	1    4700 4100
@@
 F 0 "C6" H 4415 4146 50  0000 L CNN
 F 1 "0.1u" H 4415 4055 50  0000 L CNN
-F 2 "" H 4338 3950 50  0001 C CNN
+F 2 "Capacitor_THT:C_Rect_L4.0mm_W2.5mm_P2.50mm" H 4338 3950 50  0001 C CNN
 F 3 "~" H 4300 4100 50  0001 C CNN
 	1    4300 4100
@@
 F 0 "J3" V 4746 5148 50  0000 L CNN
 F 1 "Conn_01x03_Female" V 5050 4650 50  0000 L CNN
-F 2 "" H 4900 5000 50  0001 C CNN
+F 2 "Connector_PinHeader_1.27mm:PinHeader_1x03_P1.27mm_Vertical" H 4900 5000 50  0001 C CNN
 F 3 "~" H 4900 5000 50  0001 C CNN
 	1    4900 5000
@@
 F 0 "C7" H 4515 4696 50  0000 L CNN
 F 1 "0.001u" H 4515 4605 50  0000 L CNN
-F 2 "" H 4438 4500 50  0001 C CNN
+F 2 "Capacitor_THT:C_Disc_D5.0mm_W2.5mm_P5.00mm" H 4438 4500 50  0001 C CNN
 F 3 "~" H 4400 4650 50  0001 C CNN
 	1    4400 4650
@@
 F 0 "C5" H 4115 4696 50  0000 L CNN
 F 1 "0.1u" H 4115 4605 50  0000 L CNN
-F 2 "" H 4038 4500 50  0001 C CNN
+F 2 "Capacitor_THT:C_Rect_L4.0mm_W2.5mm_P2.50mm" H 4038 4500 50  0001 C CNN
 F 3 "~" H 4000 4650 50  0001 C CNN
 	1    4000 4650
@@
 	4800 4800 4400 4800
 Connection ~ 4400 4800
-$Comp
-L Connector:Conn_01x02_Female J5
-U 1 1 5DC03624
-P 10300 2350
-F 0 "J5" H 10328 2326 50  0000 L CNN
-F 1 "Conn_01x02_Female" H 10200 2150 50  0000 L CNN
-F 2 "" H 10300 2350 50  0001 C CNN
-F 3 "~" H 10300 2350 50  0001 C CNN
-	1    10300 2350
-	1    0    0    -1
-$EndComp
-Text Notes 10650 2450 2    50   ~ 0
+Text Notes 10450 2600 2    50   ~ 0
 Motor
 Wire Wire Line
@@
 	10100 2650 10100 2450
 $Comp
-L Connector:USB_A J6
-U 1 1 5DC09B94
-P 10550 4750
-F 0 "J6" H 10320 4739 50  0000 R CNN
-F 1 "USB_A" H 10320 4648 50  0000 R CNN
-F 2 "" H 10700 4700 50  0001 C CNN
-F 3 " ~" H 10700 4700 50  0001 C CNN
-	1    10550 4750
-	-1   0    0    -1
-$EndComp
-$Comp
 L power:GND #PWR0120
 U 1 1 5DC0C0AA
-P 10650 5250
-F 0 "#PWR0120" H 10650 5000 50  0001 C CNN
-F 1 "GND" H 10655 5077 50  0000 C CNN
-F 2 "" H 10650 5250 50  0001 C CNN
-F 3 "" H 10650 5250 50  0001 C CNN
-	1    10650 5250
-	1    0    0    -1
-$EndComp
-Wire Wire Line
-	10650 5250 10650 5200
-Wire Wire Line
-	10550 5150 10550 5200
-Wire Wire Line
-	10550 5200 10650 5200
-Connection ~ 10650 5200
-Wire Wire Line
-	10650 5200 10650 5150
+P 10250 4750
+F 0 "#PWR0120" H 10250 4500 50  0001 C CNN
+F 1 "GND" H 10255 4577 50  0000 C CNN
+F 2 "" H 10250 4750 50  0001 C CNN
+F 3 "" H 10250 4750 50  0001 C CNN
+	1    10250 4750
+	1    0    0    -1
+$EndComp
 Wire Wire Line
 	10250 4550 10000 4550
 Connection ~ 10000 4550
-NoConn ~ 10250 4750
-NoConn ~ 10250 4850
 $Comp
 L Connector:Conn_01x06_Female J2
@@
 F 0 "J2" H 1092 3185 50  0000 C CNN
 F 1 "Conn_01x06_Female" H 1092 3094 50  0000 C CNN
-F 2 "" H 1200 2800 50  0001 C CNN
+F 2 "Connector_PinHeader_1.27mm:PinHeader_1x06_P1.27mm_Vertical" H 1200 2800 50  0001 C CNN
 F 3 "~" H 1200 2800 50  0001 C CNN
 	1    1200 2800
@@
 F 0 "C3" H 2865 1946 50  0000 L CNN
 F 1 "0.1u" H 2865 1855 50  0000 L CNN
-F 2 "" H 2788 1750 50  0001 C CNN
+F 2 "Capacitor_THT:C_Rect_L4.0mm_W2.5mm_P2.50mm" H 2788 1750 50  0001 C CNN
 F 3 "~" H 2750 1900 50  0001 C CNN
 	1    2750 1900
@@
 F 0 "C4" H 3265 1946 50  0000 L CNN
 F 1 "0.001u" H 3265 1855 50  0000 L CNN
-F 2 "" H 3188 1750 50  0001 C CNN
+F 2 "Capacitor_THT:C_Disc_D5.0mm_W2.5mm_P5.00mm" H 3188 1750 50  0001 C CNN
 F 3 "~" H 3150 1900 50  0001 C CNN
 	1    3150 1900
@@
 F 0 "C1" H 1315 1946 50  0000 L CNN
 F 1 "0.1u" H 1315 1855 50  0000 L CNN
-F 2 "" H 1238 1750 50  0001 C CNN
+F 2 "Capacitor_THT:C_Rect_L4.0mm_W2.5mm_P2.50mm" H 1238 1750 50  0001 C CNN
 F 3 "~" H 1200 1900 50  0001 C CNN
 	1    1200 1900
@@
 F 0 "C2" H 1715 1946 50  0000 L CNN
 F 1 "0.001u" H 1715 1855 50  0000 L CNN
-F 2 "" H 1638 1750 50  0001 C CNN
+F 2 "Capacitor_THT:C_Disc_D5.0mm_W2.5mm_P5.00mm" H 1638 1750 50  0001 C CNN
 F 3 "~" H 1600 1900 50  0001 C CNN
 	1    1600 1900
@@
 F 0 "J1" V 1046 1198 50  0000 L CNN
 F 1 "Conn_01x02_Female" H 1000 1350 50  0000 L CNN
-F 2 "" H 1200 1150 50  0001 C CNN
+F 2 "Connector_PinHeader_1.27mm:PinHeader_1x02_P1.27mm_Vertical" H 1200 1150 50  0001 C CNN
 F 3 "~" H 1200 1150 50  0001 C CNN
 	1    1200 1150
@@
 	1    0    0    -1
 $EndComp
+$Comp
+L Connector:Conn_01x03_Male J4
+U 1 1 5DB62F83
+P 5800 2850
+F 0 "J4" H 5772 2874 50  0000 R CNN
+F 1 "Conn_01x03_Male" H 5772 2783 50  0000 R CNN
+F 2 "Connector_PinHeader_1.27mm:PinHeader_1x03_P1.27mm_Vertical" H 5800 2850 50  0001 C CNN
+F 3 "~" H 5800 2850 50  0001 C CNN
+	1    5800 2850
+	-1   0    0    -1
+$EndComp
+Wire Wire Line
+	10250 4650 10250 4750
+$Comp
+L Connector:Screw_Terminal_01x02 J6
+U 1 1 5DB6AD53
+P 10450 4550
+F 0 "J6" H 10530 4542 50  0000 L CNN
+F 1 "Screw_Terminal_01x02" H 10100 4700 50  0000 L CNN
+F 2 "auto-garden:Phoenix Contact COMBICON PTSA" H 10450 4550 50  0001 C CNN
+F 3 "~" H 10450 4550 50  0001 C CNN
+	1    10450 4550
+	1    0    0    -1
+$EndComp
+Text Notes 10400 4800 0    50   ~ 0
+USB LED
+$Comp
+L Connector:Screw_Terminal_01x02 J5
+U 1 1 5DB70A1A
+P 10300 2350
+F 0 "J5" H 10380 2342 50  0000 L CNN
+F 1 "Screw_Terminal_01x02" H 9950 2500 50  0000 L CNN
+F 2 "auto-garden:Phoenix Contact COMBICON PTSA" H 10300 2350 50  0001 C CNN
+F 3 "~" H 10300 2350 50  0001 C CNN
+	1    10300 2350
+	1    0    0    -1
+$EndComp

Commit message: Finsihed board layout
Parts:
- removed U1: AP2127R-3.3, Package_TO_SOT_SMD:SOT-89-3, symbol auto-garden:AP2127R-3.3
- added U1: MCP1702-3302E_TO92-3, Package_TO_SOT_THT:TO-92, symbol auto-garden:MCP1702-3302E_TO92-3
Connections:
- net +3V3: now also U1.3 (VO)
- net +5V: now also U1.2 (VI)
- net GND: now also U1.1 (GND)
- net ~P1: now also J4.2 (Pin_2), R1.2; no longer Q1.2 (G), Q2.2 (G), R2.2
- removed net P2: J2.2 (Pin_2), J4.2 (Pin_2), R1.2
- net P3_CLK renamed P2_CLK
- net P2_CLK: now also J2.2 (Pin_2); no longer J2.3 (Pin_3)
- net P4_data renamed P3_data
- net P3_data: now also J2.3 (Pin_3); no longer J2.4 (Pin_4)
- net P5_~CS renamed P4_~CS
- net P4_~CS: now also J2.4 (Pin_4); no longer J2.5 (Pin_5)
- new net ~P5: J2.5 (Pin_5), Q1.2 (G), Q2.2 (G), R2.2
Changed lines of the file:
@@
 	8050 2900 8050 2750
 Text GLabel 7800 2350 0    50   Input ~ 0
-~P1
+~P5
 Wire Wire Line
 	8050 2350 7800 2350
@@
 Connection ~ 5300 2200
 Text GLabel 5000 2850 0    50   Input ~ 0
-P2
+~P1
 Wire Wire Line
 	5000 2850 5300 2850
@@
 Connection ~ 5500 4700
 Text GLabel 6300 4500 2    50   Input ~ 0
-P3_CLK
+P2_CLK
 Text GLabel 6650 4600 2    50   Input ~ 0
-P4_data
+P3_data
 Text GLabel 7050 4700 2    50   Input ~ 0
-P5_~CS
+P4_~CS
 Wire Wire Line
 	6300 4500 6100 4500
@@
 ~P1
 Text GLabel 1850 2700 2    50   Input ~ 0
-P2
-Text GLabel 2000 2800 2    50   Input ~ 0
-P3_CLK
-Text GLabel 2000 2900 2    50   Input ~ 0
-P4_data
-Text GLabel 2350 3000 2    50   Input ~ 0
-P5_~CS
-Text GLabel 2650 3100 2    50   Input ~ 0
-~P6
+P2_CLK
+Text GLabel 2200 2800 2    50   Input ~ 0
+P3_data
+Text GLabel 2550 2900 2    50   Input ~ 0
+P4_~CS
+Text GLabel 2850 3000 2    50   Input ~ 0
+~P5
 Wire Wire Line
 	1700 2600 1400 2600
@@
 	1400 2700 1850 2700
 Wire Wire Line
-	1400 2800 2000 2800
-Wire Wire Line
-	2000 2900 1400 2900
-Wire Wire Line
-	1400 3000 2350 3000
-Wire Wire Line
-	1400 3100 2650 3100
-$Comp
-L auto-garden:AP2127R-3.3 U1
-U 1 1 5DC4D600
-P 2200 1750
-F 0 "U1" H 2200 1992 50  0000 C CNN
-F 1 "AP2127R-3.3" H 2200 1901 50  0000 C CNN
-F 2 "Package_TO_SOT_SMD:SOT-89-3" H 2200 1950 50  0001 C CNN
-F 3 "https://www.diodes.com/assets/Datasheets/AP2127.pdf" H 2200 1700 50  0001 C CNN
-	1    2200 1750
-	1    0    0    -1
-$EndComp
+	1400 2800 2200 2800
+Wire Wire Line
+	2550 2900 1400 2900
+Wire Wire Line
+	1400 3000 2850 3000
+Wire Wire Line
+	1400 3100 3000 3100
 $Comp
 L power:+5V #PWR0121
@@
 	1    0    0    -1
 $EndComp
+$Comp
+L auto-garden:MCP1702-3302E_TO92-3 U1
+U 1 1 5DB85411
+P 2200 1750
+F 0 "U1" H 2200 1992 50  0000 C CNN
+F 1 "MCP1702-3302E_TO92-3" H 2200 1901 50  0000 C CNN
+F 2 "Package_TO_SOT_THT:TO-92" H 2200 1950 50  0001 C CNN
+F 3 "http://ww1.microchip.com/downloads/en/DeviceDoc/20005122B.pdf" H 2200 1700 50  0001 C CNN
+	1    2200 1750
+	1    0    0    -1
+$EndComp
+Text GLabel 3000 3100 2    50   Input ~ 0
+~P6
 $EndSCHEMATC

Commit message: editted pin header footprints
Parts:
- J1: footprint Connector_PinHeader_1.27mm:PinHeader_1x02_P1.27mm_Vertical -> Connector_PinSocket_2.54mm:PinSocket_1x02_P2.54mm_Horizontal
- J2: footprint Connector_PinHeader_1.27mm:PinHeader_1x06_P1.27mm_Vertical -> Connector_PinSocket_2.54mm:PinSocket_1x06_P2.54mm_Vertical
- J3: footprint Connector_PinHeader_1.27mm:PinHeader_1x03_P1.27mm_Vertical -> Connector_PinSocket_2.54mm:PinSocket_1x03_P2.54mm_Vertical
- J4: footprint Connector_PinHeader_1.27mm:PinHeader_1x03_P1.27mm_Vertical -> Connector_PinHeader_2.54mm:PinHeader_1x03_P2.54mm_Vertical
Changed lines of the file:
@@
 F 0 "J3" V 4746 5148 50  0000 L CNN
 F 1 "Conn_01x03_Female" V 5050 4650 50  0000 L CNN
-F 2 "Connector_PinHeader_1.27mm:PinHeader_1x03_P1.27mm_Vertical" H 4900 5000 50  0001 C CNN
+F 2 "Connector_PinSocket_2.54mm:PinSocket_1x03_P2.54mm_Vertical" H 4900 5000 50  0001 C CNN
 F 3 "~" H 4900 5000 50  0001 C CNN
 	1    4900 5000
@@
 F 0 "J2" H 1092 3185 50  0000 C CNN
 F 1 "Conn_01x06_Female" H 1092 3094 50  0000 C CNN
-F 2 "Connector_PinHeader_1.27mm:PinHeader_1x06_P1.27mm_Vertical" H 1200 2800 50  0001 C CNN
+F 2 "Connector_PinSocket_2.54mm:PinSocket_1x06_P2.54mm_Vertical" H 1200 2800 50  0001 C CNN
 F 3 "~" H 1200 2800 50  0001 C CNN
 	1    1200 2800
@@
 F 0 "J1" V 1046 1198 50  0000 L CNN
 F 1 "Conn_01x02_Female" H 1000 1350 50  0000 L CNN
-F 2 "Connector_PinHeader_1.27mm:PinHeader_1x02_P1.27mm_Vertical" H 1200 1150 50  0001 C CNN
+F 2 "Connector_PinSocket_2.54mm:PinSocket_1x02_P2.54mm_Horizontal" H 1200 1150 50  0001 C CNN
 F 3 "~" H 1200 1150 50  0001 C CNN
 	1    1200 1150
@@
 F 0 "J4" H 5772 2874 50  0000 R CNN
 F 1 "Conn_01x03_Male" H 5772 2783 50  0000 R CNN
-F 2 "Connector_PinHeader_1.27mm:PinHeader_1x03_P1.27mm_Vertical" H 5800 2850 50  0001 C CNN
+F 2 "Connector_PinHeader_2.54mm:PinHeader_1x03_P2.54mm_Vertical" H 5800 2850 50  0001 C CNN
 F 3 "~" H 5800 2850 50  0001 C CNN
 	1    5800 2850

Commit message: rerouted with new pin headers
Parts:
- J1: footprint Connector_PinSocket_2.54mm:PinSocket_1x02_P2.54mm_Horizontal -> Connector_PinSocket_2.54mm:PinSocket_1x02_P2.54mm_Vertical
Changed lines of the file:
@@
 F 0 "J1" V 1046 1198 50  0000 L CNN
 F 1 "Conn_01x02_Female" H 1000 1350 50  0000 L CNN
-F 2 "Connector_PinSocket_2.54mm:PinSocket_1x02_P2.54mm_Horizontal" H 1200 1150 50  0001 C CNN
+F 2 "Connector_PinSocket_2.54mm:PinSocket_1x02_P2.54mm_Vertical" H 1200 1150 50  0001 C CNN
 F 3 "~" H 1200 1150 50  0001 C CNN
 	1    1200 1150
